File: hardware/fydp/Analog Multiplier 2.kicad_sch (KiCad schematic)
At the start: 21 parts, among them J8 Conn_01x02_Pin, U1 LTC2630ISC6-LZ8-TRMPBF, U3 SN74LVC1G3157DCKR, U4 LTC2630ISC6-LZ8-TRMPBF, U5 SN74LVC1G3157DCKR, U6 AD633ARZ-R7

Commit message: Remove 2 channels of multiplier and change ADC
Parts:
- removed C1, C16: 0.01uF, Capacitor_SMD:C_0805_2012Metric, symbol Device:C
- removed C11, C14, C20, C23, C5, C8: 0.1uF, Capacitor_SMD:C_0805_2012Metric, symbol Device:C
- removed J8: Conn_01x02_Pin, Connector_PinHeader_2.54mm:PinHeader_1x02_P2.54mm_Vertical, symbol Connector:Conn_01x02_Pin
- removed R1, R2, R3, R4: 1K, Resistor_SMD:R_0805_2012Metric, symbol Device:R
- removed R52 (x2): 100, Resistor_SMD:R_0805_2012Metric, symbol Device:R
- removed U1, U4: LTC2630ISC6-LZ8-TRMPBF, Package_TO_SOT_SMD:SOT-363_SC-70-6_Handsoldering, symbol LTC2630ISC6-LZ8#TRMPBF:LTC2630ISC6-LZ8-TRMPBF
- removed U3, U5: SN74LVC1G3157DCKR, Package_TO_SOT_SMD:SOT-23-6_Handsoldering, symbol SN74LVC1G3157DCKR:SN74LVC1G3157DCKR
- removed U6 (x2): AD633ARZ-R7, fydp:R_8_ADI, symbol AD633ARZ-R7:AD633ARZ-R7
Other:
- note removed: "ANALOG MULTIPLIER (2/8)"
- note removed: "ANALOG SWITCH SELECT GPIO TO FPGA *THESE ARE 5V GPIOS*"
- note removed: "When S is HIGH, B2 passes When S is LOW, B1 passes"
- note removed: "[1,3]"
- note removed: "[1,4]"
