File: hardware/fydp/DAC Inputs.kicad_sch (KiCad schematic)
At the start: 11 parts, among them J14 Conn_01x02_Pin, U1 LTC2630ISC6-LZ8-TRMPBF

Commit message: Pushing laptop changes
Parts:
- U1: value LTC2630ISC6-LZ8-TRMPBF -> LTC2630ISC6-HZ12#TRMPBF; Comment 8 Bit Digital to Analog Converter 1 SC-70-6 -> 12 Bit Digital to Analog Converter 1 SC-70-6; MPN LTC2630ISC6-LZ8#TRMPBF -> LTC2630ISC6-HZ12#TRMPBF
Changed lines of the file:
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@@
       (effects (font (size 1.524 1.524)))
     )
-    (property "Value" "LTC2630ISC6-LZ8-TRMPBF" (at 209.55 101.6 0)
+    (property "Value" "LTC2630ISC6-HZ12#TRMPBF" (at 209.55 101.6 0)
       (effects (font (size 1.524 1.524)))
     )
@@
       (effects (font (size 1.27 1.27) italic) hide)
     )
-    (property "Comment" "8 Bit Digital to Analog Converter 1 SC-70-6" (at 186.69 109.22 0)
-      (effects (font (size 1.27 1.27)) hide)
-    )
-    (property "MPN" "LTC2630ISC6-LZ8#TRMPBF" (at 186.69 109.22 0)
+    (property "Comment" "12 Bit Digital to Analog Converter 1 SC-70-6" (at 186.69 109.22 0)
+      (effects (font (size 1.27 1.27)) hide)
+    )
+    (property "MPN" "LTC2630ISC6-HZ12#TRMPBF" (at 186.69 109.22 0)
       (effects (font (size 1.27 1.27)) hide)
     )
@@
       (effects (font (size 1.524 1.524)))
     )
-    (property "Value" "LTC2630ISC6-LZ8-TRMPBF" (at 95.25 101.6 0)
+    (property "Value" "LTC2630ISC6-HZ12#TRMPBF" (at 95.25 101.6 0)
       (effects (font (size 1.524 1.524)))
     )
@@
       (effects (font (size 1.27 1.27) italic) hide)
     )
-    (property "Comment" "8 Bit Digital to Analog Converter 1 SC-70-6" (at 72.39 109.22 0)
-      (effects (font (size 1.27 1.27)) hide)
-    )
-    (property "MPN" "LTC2630ISC6-LZ8#TRMPBF" (at 72.39 109.22 0)
+    (property "Comment" "12 Bit Digital to Analog Converter 1 SC-70-6" (at 72.39 109.22 0)
+      (effects (font (size 1.27 1.27)) hide)
+    )
+    (property "MPN" "LTC2630ISC6-HZ12#TRMPBF" (at 72.39 109.22 0)
       (effects (font (size 1.27 1.27)) hide)
     )
@@
       (effects (font (size 1.524 1.524)))
     )
-    (property "Value" "LTC2630ISC6-LZ8-TRMPBF" (at 209.55 43.18 0)
+    (property "Value" "LTC2630ISC6-HZ12#TRMPBF" (at 209.55 43.18 0)
       (effects (font (size 1.524 1.524)))
     )
@@
       (effects (font (size 1.27 1.27) italic) hide)
     )
-    (property "Comment" "8 Bit Digital to Analog Converter 1 SC-70-6" (at 186.69 50.8 0)
-      (effects (font (size 1.27 1.27)) hide)
-    )
-    (property "MPN" "LTC2630ISC6-LZ8#TRMPBF" (at 186.69 50.8 0)
+    (property "Comment" "12 Bit Digital to Analog Converter 1 SC-70-6" (at 186.69 50.8 0)
+      (effects (font (size 1.27 1.27)) hide)
+    )
+    (property "MPN" "LTC2630ISC6-HZ12#TRMPBF" (at 186.69 50.8 0)
       (effects (font (size 1.27 1.27)) hide)
     )
@@
       (effects (font (size 1.524 1.524)))
     )
-    (property "Value" "LTC2630ISC6-LZ8-TRMPBF" (at 95.25 43.18 0)
+    (property "Value" "LTC2630ISC6-HZ12#TRMPBF" (at 95.25 43.18 0)
       (effects (font (size 1.524 1.524)))
     )
@@
       (effects (font (size 1.27 1.27) italic) hide)
     )
-    (property "Comment" "8 Bit Digital to Analog Converter 1 SC-70-6" (at 72.39 50.8 0)
-      (effects (font (size 1.27 1.27)) hide)
-    )
-    (property "MPN" "LTC2630ISC6-LZ8#TRMPBF" (at 72.39 50.8 0)
-      (effects (font (size 1.27 1.27)) hide)
-    )
+    (property "Comment" "12 Bit Digital to Analog Converter 1 SC-70-6" (at 72.39 50.8 0)
+      (effects (font (size 1.27 1.27)) hide)
+    )
+    (property "MPN" "LTC2630ISC6-HZ12#TRMPBF" (at 72.39 50.8 0)
+      (effects (font (size 1.27 1.27)) hide)
+    )

Commit message: Fixed footprints
Parts:
- J14: value Conn_01x02_Pin -> TSW-102-07-G-S
Changed lines of the file:
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@@
       (effects (font (size 1.27 1.27)))
     )
-    (property "Value" "Conn_01x02_Pin" (at 53.975 166.37 0)
+    (property "Value" "TSW-102-07-G-S" (at 53.975 166.37 0)
       (effects (font (size 1.27 1.27)))
     )
