File: hardware/fydp/DECODER 2.kicad_sch (KiCad schematic)
At the start: 42 parts, among them J11 Conn_01x04_Pin, J12 Conn_01x04_Pin, U5 74HC154D

Commit message: Updating BOM some more
Parts:
- J11, J12: Comment (none) -> Connector Header Through Hole 4 position 0.100" (2.54mm); MPN (none) -> TSW-104-07-G-S
- U5: MPN (none) -> 74HC154D
Changed lines of the file:
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@@
       (effects (font (size 1.27 1.27) italic) hide)
+    )
+    (property "MPN" "74HC154D" (at 97.79 82.55 0)
+      (effects (font (size 1.27 1.27)) hide)
     )
     (pin "1")
@@
       (effects (font (size 1.27 1.27)) hide)
     )
-    (property "Datasheet" "~" (at 156.21 50.8 0)
+    (property "Datasheet" "https://suddendocs.samtec.com/catalog_english/tsw_th.pdf" (at 156.21 50.8 0)
+      (effects (font (size 1.27 1.27)) hide)
+    )
+    (property "Comment" "Connector Header Through Hole 4 position 0.100\" (2.54mm)" (at 156.21 50.8 0)
+      (effects (font (size 1.27 1.27)) hide)
+    )
+    (property "MPN" "TSW-104-07-G-S" (at 156.21 50.8 0)
       (effects (font (size 1.27 1.27)) hide)
     )
@@
       (effects (font (size 1.27 1.27)) hide)
     )
-    (property "Datasheet" "~" (at 276.86 107.95 0)
-      (effects (font (size 1.27 1.27)) hide)
-    )
+    (property "Datasheet" "https://suddendocs.samtec.com/catalog_english/tsw_th.pdf" (at 276.86 107.95 0)
+      (effects (font (size 1.27 1.27)) hide)
+    )
+    (property "Comment" "Connector Header Through Hole 4 position 0.100\" (2.54mm)" (at 276.86 107.95 0)
+      (effects (font (size 1.27 1.27)) hide)
+    )
+    (property "MPN" "TSW-104-07-G-S" (at 276.86 107.95 0)
+      (effects (font (size 1.27 1.27)) hide)
+    )

Commit message: Pushing laptop changes
Parts:
- U5: value 74HC154D -> CD74HC154M96; Comment (none) -> Decoder/Demultiplexer 1 x 4:16 24-SOIC; LCSC (none) -> C2832236; MPN 74HC154D -> CD74HC154M96
Changed lines of the file:
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@@
       (effects (font (size 1.524 1.524)))
     )
-    (property "Value" "74HC154D" (at 128.27 74.93 0)
+    (property "Value" "CD74HC154M96" (at 128.27 74.93 0)
       (effects (font (size 1.524 1.524)))
     )
@@
       (effects (font (size 1.27 1.27) italic) hide)
     )
-    (property "Datasheet" "74HC154D" (at 97.79 82.55 0)
+    (property "Datasheet" "https://www.ti.com/general/docs/suppproductinfo.tsp?distId=10&gotoUrl=https%3A%2F%2Fwww.ti.com%2Flit%2Fgpn%2Fcd74hc154" (at 97.79 82.55 0)
       (effects (font (size 1.27 1.27) italic) hide)
     )
-    (property "MPN" "74HC154D" (at 97.79 82.55 0)
+    (property "MPN" "CD74HC154M96" (at 97.79 82.55 0)
       (effects (font (size 1.27 1.27)) hide)
     )
+    (property "Comment" "Decoder/Demultiplexer 1 x 4:16 24-SOIC" (at 97.79 82.55 0)
+      (effects (font (size 1.27 1.27)) hide)
+    )
+    (property "LCSC" "C2832236" (at 97.79 82.55 0)
+      (effects (font (size 1.27 1.27)) hide)
+    )

Commit message: Fixed footprints
Parts:
- J11, J12: value Conn_01x04_Pin -> TSW-104-07-G-S
Changed lines of the file:
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@@
       (effects (font (size 1.27 1.27)))
     )
-    (property "Value" "Conn_01x04_Pin" (at 155.575 45.72 0)
+    (property "Value" "TSW-104-07-G-S" (at 155.575 45.72 0)
       (effects (font (size 1.27 1.27)))
     )
@@
       (effects (font (size 1.27 1.27)))
     )
-    (property "Value" "Conn_01x04_Pin" (at 276.225 102.87 0)
-      (effects (font (size 1.27 1.27)))
-    )
+    (property "Value" "TSW-104-07-G-S" (at 276.225 102.87 0)
+      (effects (font (size 1.27 1.27)))
+    )
