File: hardware/fydp/Decoder 1.kicad_sch (KiCad schematic)
At the start: 25 parts, among them J4 Conn_01x08_Pin, U4 74HC139N

Commit message: Pushing laptop changes
Parts:
- U4: value 74HC139N -> 74HC139D,653; Comment (none) -> Decoder/Demultiplexer 1 x 2:4 16-SO; LCSC (none) -> C5603; MPN 74HC139N -> 74HC139D,653
Changed lines of the file:
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@@
       (effects (font (size 1.524 1.524)))
     )
-    (property "Value" "74HC139N" (at 151.13 92.71 0)
+    (property "Value" "74HC139D,653" (at 151.13 92.71 0)
       (effects (font (size 1.524 1.524)))
     )
@@
       (effects (font (size 1.27 1.27) italic) hide)
     )
-    (property "Datasheet" "74HC139N" (at 181.61 100.33 0)
+    (property "Datasheet" "https://assets.nexperia.com/documents/data-sheet/74HC_HCT139.pdf" (at 181.61 100.33 0)
       (effects (font (size 1.27 1.27) italic) hide)
     )
-    (property "MPN" "74HC139N" (at 181.61 100.33 0)
+    (property "MPN" "74HC139D,653" (at 181.61 100.33 0)
       (effects (font (size 1.27 1.27)) hide)
     )
+    (property "Comment" "Decoder/Demultiplexer 1 x 2:4 16-SO" (at 181.61 100.33 0)
+      (effects (font (size 1.27 1.27)) hide)
+    )
+    (property "LCSC" "C5603" (at 181.61 100.33 0)
+      (effects (font (size 1.27 1.27)) hide)
+    )

Commit message: Fixed footprints
Parts:
- J4: value Conn_01x08_Pin -> TSW-108-07-G-S
Changed lines of the file:
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@@
       (effects (font (size 1.27 1.27)) (justify right))
     )
-    (property "Value" "Conn_01x08_Pin" (at 267.97 57.15 0)
+    (property "Value" "TSW-108-07-G-S" (at 267.97 57.15 0)
       (effects (font (size 1.27 1.27)) (justify right))
     )
