File: hardware/fydp/USBC_Receptacle.kicad_sch (KiCad schematic)
At the start: 14 parts, among them J1 1054500101, J2 Conn_01x02_Pin, J3 Conn_01x02_Pin

Commit message: Finished layout
Parts:
- added J10, J13, J8, J9: 5011, 5011:CONN1_5011_KEY, symbol 5011:5011
Connections:
- net GND: now also J10.1, J13.1, J8.1, J9.1
Changed lines of the file:
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@@
   (junction (at 224.79 54.61) (diameter 0) (color 0 0 0 0)
   )
+  (junction (at 116.84 171.45) (diameter 0) (color 0 0 0 0)
+  )
   (junction (at 146.05 54.61) (diameter 0) (color 0 0 0 0)
   )
   (junction (at 39.37 179.07) (diameter 0) (color 0 0 0 0)
   )
+  (junction (at 116.84 163.83) (diameter 0) (color 0 0 0 0)
+  )
   (junction (at 213.36 54.61) (diameter 0) (color 0 0 0 0)
   )
@@
   )
   (junction (at 140.97 105.41) (diameter 0) (color 0 0 0 0)
+  )
+  (junction (at 116.84 156.21) (diameter 0) (color 0 0 0 0)
   )
   (junction (at 170.18 54.61) (diameter 0) (color 0 0 0 0)
@@
     (stroke (width 0) (type default))
   )
+  (wire (pts (xy 116.84 171.45) (xy 116.84 172.72))
+    (stroke (width 0) (type default))
+  )
+  (wire (pts (xy 116.84 156.21) (xy 118.11 156.21))
+    (stroke (width 0) (type default))
+  )
   (wire (pts (xy 53.34 177.8) (xy 53.34 179.07))
     (stroke (width 0) (type default))
@@
     (stroke (width 0) (type default))
   )
+  (wire (pts (xy 116.84 156.21) (xy 116.84 163.83))
+    (stroke (width 0) (type default))
+  )
   (wire (pts (xy 39.37 179.07) (xy 39.37 180.34))
     (stroke (width 0) (type default))
@@
     (stroke (width 0) (type default))
   )
+  (wire (pts (xy 116.84 148.59) (xy 116.84 156.21))
+    (stroke (width 0) (type default))
+  )
   (wire (pts (xy 130.81 46.99) (xy 128.27 46.99))
     (stroke (width 0) (type default))
@@
     (stroke (width 0) (type default))
   )
+  (wire (pts (xy 116.84 163.83) (xy 118.11 163.83))
+    (stroke (width 0) (type default))
+  )
   (wire (pts (xy 146.05 54.61) (xy 156.21 54.61))
     (stroke (width 0) (type default))
@@
     (stroke (width 0) (type default))
   )
+  (wire (pts (xy 116.84 171.45) (xy 118.11 171.45))
+    (stroke (width 0) (type default))
+  )
   (wire (pts (xy 201.93 54.61) (xy 213.36 54.61))
     (stroke (width 0) (type default))
@@
     (stroke (width 0) (type default))
   )
+  (wire (pts (xy 116.84 163.83) (xy 116.84 171.45))
+    (stroke (width 0) (type default))
+  )
   (wire (pts (xy 140.97 66.04) (xy 140.97 105.41))
+    (stroke (width 0) (type default))
+  )
+  (wire (pts (xy 118.11 148.59) (xy 116.84 148.59))
     (stroke (width 0) (type default))
   )
@@
     )
   )
+  (symbol (lib_id "power:GND") (at 116.84 172.72 0) (unit 1)
+    (in_bom yes) (on_board yes) (dnp no) (fields_autoplaced)
+    (property "Reference" "#PWR031" (at 116.84 179.07 0)
+      (effects (font (size 1.27 1.27)) hide)
+    )
+    (property "Value" "GND" (at 116.84 177.8 0)
+      (effects (font (size 1.27 1.27)))
+    )
+    (property "Footprint" "" (at 116.84 172.72 0)
+      (effects (font (size 1.27 1.27)) hide)
+    )
+    (property "Datasheet" "" (at 116.84 172.72 0)
+      (effects (font (size 1.27 1.27)) hide)
+    )
+    (pin "1")
+    (instances
+      (project "fydp"
+        (path "/2d5d1aad-2c7d-465e-90ef-822dec61a05e/fa9eb183-9fe8-4a28-a113-cdc4462de8b4"
+          (reference "#PWR031") (unit 1)
+        )
+      )
+    )
+  )
   (symbol (lib_id "power:GND") (at 201.93 64.77 0) (unit 1)
     (in_bom yes) (on_board yes) (dnp no)
@@
         (path "/2d5d1aad-2c7d-465e-90ef-822dec61a05e/fa9eb183-9fe8-4a28-a113-cdc4462de8b4"
           (reference "R98") (unit 1)
+        )
+      )
+    )
+  )
+  (symbol (lib_id "5011:5011") (at 118.11 171.45 0) (unit 1)
+    (in_bom yes) (on_board yes) (dnp no) (fields_autoplaced)
+    (property "Reference" "J13" (at 132.08 170.18 0)
+      (effects (font (size 1.524 1.524)) (justify left))
+    )
+    (property "Value" "5011" (at 132.08 172.72 0)
+      (effects (font (size 1.524 1.524)) (justify left))
+    )
+    (property "Footprint" "5011:CONN1_5011_KEY" (at 118.11 171.45 0)
+      (effects (font (size 1.27 1.27) italic) hide)
+    )
+    (property "Datasheet" "5011" (at 118.11 171.45 0)
+      (effects (font (size 1.27 1.27) italic) hide)
+    )
+    (pin "1")
+    (instances
+      (project "fydp"
+        (path "/2d5d1aad-2c7d-465e-90ef-822dec61a05e/fa9eb183-9fe8-4a28-a113-cdc4462de8b4"
+          (reference "J13") (unit 1)
         )
       )
@@
     )
   )
+  (symbol (lib_id "5011:5011") (at 118.11 156.21 0) (unit 1)
+    (in_bom yes) (on_board yes) (dnp no) (fields_autoplaced)
+    (property "Reference" "J9" (at 132.08 154.94 0)
+      (effects (font (size 1.524 1.524)) (justify left))
+    )
+    (property "Value" "5011" (at 132.08 157.48 0)
+      (effects (font (size 1.524 1.524)) (justify left))
+    )
+    (property "Footprint" "5011:CONN1_5011_KEY" (at 118.11 156.21 0)
+      (effects (font (size 1.27 1.27) italic) hide)
+    )
+    (property "Datasheet" "5011" (at 118.11 156.21 0)
+      (effects (font (size 1.27 1.27) italic) hide)
+    )
+    (pin "1")
+    (instances
+      (project "fydp"
+        (path "/2d5d1aad-2c7d-465e-90ef-822dec61a05e/fa9eb183-9fe8-4a28-a113-cdc4462de8b4"
+          (reference "J9") (unit 1)
+        )
+      )
+    )
+  )
+  (symbol (lib_id "5011:5011") (at 118.11 163.83 0) (unit 1)
+    (in_bom yes) (on_board yes) (dnp no) (fields_autoplaced)
+    (property "Reference" "J8" (at 132.08 162.56 0)
+      (effects (font (size 1.524 1.524)) (justify left))
+    )
+    (property "Value" "5011" (at 132.08 165.1 0)
+      (effects (font (size 1.524 1.524)) (justify left))
+    )
+    (property "Footprint" "5011:CONN1_5011_KEY" (at 118.11 163.83 0)
+      (effects (font (size 1.27 1.27) italic) hide)
+    )
+    (property "Datasheet" "5011" (at 118.11 163.83 0)
+      (effects (font (size 1.27 1.27) italic) hide)
+    )
+    (pin "1")
+    (instances
+      (project "fydp"
+        (path "/2d5d1aad-2c7d-465e-90ef-822dec61a05e/fa9eb183-9fe8-4a28-a113-cdc4462de8b4"
+          (reference "J8") (unit 1)
+        )
+      )
+    )
+  )
   (symbol (lib_id "power:GND") (at 224.79 64.77 0) (unit 1)
     (in_bom yes) (on_board yes) (dnp no)
@@
         )
       )
+    )
+  )
+  (symbol (lib_id "5011:5011") (at 118.11 148.59 0) (unit 1)
+    (in_bom yes) (on_board yes) (dnp no) (fields_autoplaced)
+    (property "Reference" "J10" (at 132.08 147.32 0)
+      (effects (font (size 1.524 1.524)) (justify left))
+    )
+    (property "Value" "5011" (at 132.08 149.86 0)
+      (effects (font (size 1.524 1.524)) (justify left))
+    )
+    (property "Footprint" "5011:CONN1_5011_KEY" (at 118.11 148.59 0)
+      (effects (font (size 1.27 1.27) italic) hide)
+    )
+    (property "Datasheet" "5011" (at 118.11 148.59 0)
+      (effects (font (size 1.27 1.27) italic) hide)
+    )
+    (pin "1")
+    (instances
+      (project "fydp"
+        (path "/2d5d1aad-2c7d-465e-90ef-822dec61a05e/fa9eb183-9fe8-4a28-a113-cdc4462de8b4"
+          (reference "J10") (unit 1)
+        )
+      )

Commit message: Adding JLCPCB BOM notes
Parts:
- C24: Comment (none) -> 4.7 µF ±10% 25V Ceramic Capacitor X7R 0805 (2012 Metric); LCSC (none) -> C354262; MPN (none) -> CC0805KKX7R8BB475
- F1: Comment (none) -> 500 mA 63 V AC 63 V DC Fuse Board Mount (Cartridge Style Ex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; LCSC (none) -> C206953; MPN (none) -> 0437.500WR
- J1: Comment (none) -> USB-C (USB TYPE-C) USB 3.2 Gen 2 (USB 3.1 Gen 2, Superspeed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; LCSC (none) -> C134092; MPN (none) -> 1054500101
- J10, J13, J8, J9: Comment (none) -> Black PC Test Point, Multipurpose Phosphor Bronze Silver Pl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; LCSC (none) -> C238127; MPN (none) -> 5011
- J3: Comment (none) -> 2 Position Wire to Board Terminal Block Horizontal with Boa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; LCSC (none) -> C89122; MPN (none) -> 1751248
- R97, R98: Comment (none) -> 5.1 kOhms ±0.1% 0.125W, 1/8W Chip Resistor 0805 (2012 Metri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; LCSC (none) -> C865574; MPN (none) -> RT0805BRD075K1L

Commit message: Updating BOM some more
Parts:
- J2: Comment (none) -> Connector Header Through Hole 2 position 0.100" (2.54mm); MPN (none) -> TSW-102-07-G-S
Changed lines of the file:
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@@
       (effects (font (size 1.27 1.27)) hide)
     )
-    (property "Datasheet" "~" (at 156.21 49.53 0)
+    (property "Datasheet" "https://suddendocs.samtec.com/catalog_english/tsw_th.pdf" (at 156.21 49.53 0)
       (effects (font (size 1.27 1.27)) hide)
     )
+    (property "Comment" "Connector Header Through Hole 2 position 0.100\" (2.54mm)" (at 156.21 49.53 0)
+      (effects (font (size 1.27 1.27)) hide)
+    )
+    (property "MPN" "TSW-102-07-G-S" (at 156.21 49.53 0)
+      (effects (font (size 1.27 1.27)) hide)
+    )

Commit message: Fixed footprints
Parts:
- D1: value TPD1E10B06DPYR -> CDSOD323-T05; footprint Resistor_SMD:R_0805_2012Metric -> Diode_SMD:D_SOD-323_HandSoldering; Comment (none) -> 18.3V (Typ) Clamp 17A (8/20µs) Ipp Tvs Diode Surface Mount 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; LCSC (none) -> C3706224; MPN (none) -> CDSOD323-T05
- J2: value Conn_01x02_Pin -> TSW-102-07-G-S
- J3: value Conn_01x02_Pin -> 1751248
Changed lines of the file:
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@@
       (effects (font (size 1.27 1.27)))
     )
-    (property "Value" "Conn_01x02_Pin" (at 158.75 46.99 90)
+    (property "Value" "TSW-102-07-G-S" (at 158.75 46.99 90)
       (effects (font (size 1.27 1.27)))
     )
@@
       (effects (font (size 1.27 1.27)) (justify left))
     )
-    (property "Value" "Conn_01x02_Pin" (at 168.91 46.99 90)
+    (property "Value" "1751248" (at 168.91 46.99 90)
       (effects (font (size 1.27 1.27)) (justify left))
     )
@@
       (effects (font (size 1.524 1.524)) (justify left))
     )
-    (property "Value" "TPD1E10B06DPYR" (at 194.31 74.676 90)
-      (effects (font (size 1.524 1.524)) (justify left))
-    )
-    (property "Footprint" "Resistor_SMD:R_0805_2012Metric" (at 190.5 57.15 0)
-      (effects (font (size 1.27 1.27) italic) hide)
-    )
-    (property "Datasheet" "TPD1E10B06DPYR" (at 194.31 72.39 0)
-      (effects (font (size 1.27 1.27) italic) hide)
-    )
-    (pin "1")
+    (property "Value" "CDSOD323-T05" (at 194.31 74.676 90)
+      (effects (font (size 1.524 1.524)) (justify left))
+    )
+    (property "Footprint" "Diode_SMD:D_SOD-323_HandSoldering" (at 190.5 57.15 0)
+      (effects (font (size 1.27 1.27) italic) hide)
+    )
+    (property "Datasheet" "https://www.bourns.com/docs/Product-Datasheets/CDSOD323-TxxC.PDF" (at 194.31 72.39 0)
+      (effects (font (size 1.27 1.27) italic) hide)
+    )
+    (property "Comment" "18.3V (Typ) Clamp 17A (8/20µs) Ipp Tvs Diode Surface Mount SOD-323" (at 190.5 57.15 0)
+      (effects (font (size 1.27 1.27)) hide)
+    )
+    (property "LCSC" "C3706224" (at 190.5 57.15 0)
+      (effects (font (size 1.27 1.27)) hide)
+    )
+    (property "MPN" "CDSOD323-T05" (at 190.5 57.15 0)
+      (effects (font (size 1.27 1.27)) hide)
+    )
+    (pin "1")

Commit message: Production underway, Mingze is tired
Parts:
- J3: footprint TerminalBlock_Phoenix:TerminalBlock_Phoenix_PT-1,5-2-3.5-H_1x02_P3.50mm_Horizontal -> 1751248:CONN_1751248_PXC
Changed lines of the file:
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@@
       (effects (font (size 1.27 1.27)) (justify left))
     )
-    (property "Footprint" "TerminalBlock_Phoenix:TerminalBlock_Phoenix_PT-1,5-2-3.5-H_1x02_P3.50mm_Horizontal" (at 172.72 49.53 0)
+    (property "Footprint" "1751248:CONN_1751248_PXC" (at 172.72 49.53 0)
       (effects (font (size 1.27 1.27)) hide)
     )
